File: eagle/schematic/plugstrip.brd (EAGLE design)
At the start: 100 x 80 mm, 10 parts, among them J1 213598-2, U1 Hall Effect

Commit message: update board
Parts:
- RELAY1: value (none) -> RELAY
- U2: value (none) -> ADC
Changed lines of the file:
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@@
 <element name="R2" library="jackIdd" package="0411/15" value="10K" x="-21.59" y="60.96"/>
 <element name="R3" library="jackIdd" package="0411/15" value="" x="-38.1" y="60.96"/>
-<element name="RELAY1" library="iddproject" package="G5RL-1A-E-HR" value="" x="-30.48" y="40.64"/>
+<element name="RELAY1" library="iddproject" package="G5RL-1A-E-HR" value="RELAY" x="-30.48" y="40.64"/>
 <element name="U1" library="iddproject" package="ACS711" value="Hall Effect" x="-52.07" y="41.91"/>
-<element name="U2" library="iddproject" package="ADS1013" value="" x="-21.59" y="53.34"/>
+<element name="U2" library="iddproject" package="ADS1013" value="ADC" x="-21.59" y="53.34"/>
 </elements>
 <signals>

Commit message: save schematic, board
Parts:
- added C2, C3, C4: 1uF, jackIdd:C2.5-2
- added D2, D3, D4: BAT54, diode:SOT23
- added J2, J3, J4: 213598-2, con-amp:213598-2
- added Q2, Q3, Q4: (no value), jackIdd:SOT23
- added R10, R4, R7: 1K, jackIdd:0411/15
- added R11, R5, R8: 10K, jackIdd:0411/15
- added R12, R6, R9: 200K, jackIdd:0411/15
- added RELAY2, RELAY3, RELAY4: RELAY, iddproject:G5RL-1A-E-HR
- added SV2: (no value), con-lstb:MA13-1
- added U3, U5, U7: Hall Effect, iddproject:ACS711
- added U4, U6, U8: ADC, iddproject:ADS1013
- C1: value (none) -> 1uF
- R3: value (none) -> 200K
- moved C1 65.6 mm to (47.0, 69.8)
- moved D1 65.6 mm to (35.6, 71.1)
- moved J1 65.6 mm to (34.3, 33.0)
- moved Q1 65.6 mm to (29.2, 68.6)
- moved R1 65.6 mm to (19.1, 68.6)
- moved R2 65.6 mm to (41.9, 77.5)
- moved R3 65.6 mm to (25.4, 77.5)
- moved RELAY1 65.6 mm to (33.0, 57.1)
- moved U1 65.6 mm to (11.4, 58.4)
- moved U2 65.6 mm to (41.9, 69.8)
Connections:
- removed net D4: R1.1
- removed net D5: U1.P$6
- new net AC_LIVE: U1.P$3, U1.P$4, U3.P$3, U3.P$4, U5.P$3, U5.P$4, U7.P$3, U7.P$4
- new net AC_NEUTRAL: RELAY1.IN2, RELAY2.IN2, RELAY3.IN2, RELAY4.IN2
- new net D10: R7.1, SV2.10
- new net D11: SV2.11, U5.P$6
- new net D12: R10.1, SV2.12
- new net D13: SV2.13, U7.P$6
- new net D6: R1.1, SV2.6
- new net D7: SV2.7, U1.P$6
- new net D8: R4.1, SV2.8
- new net D9: SV2.9, U3.P$6
- new net N$10: SV2.2
- new net N$11: J2.2, RELAY2.IN1
- new net N$12: RELAY2.OUT2, U3.P$1, U3.P$2
- new net N$13: Q2.P$3, RELAY2.ON1
- new net N$14: Q2.P$1, R4.2, R5.2
- new net N$15: D2.1, U3.P$7
- new net N$16: C2.1, D2.3, R6.2, U4.P$4
- new net N$17: J4.3, RELAY4.OUT1
- new net N$18: J3.3, RELAY3.OUT1
- new net N$19: J3.2, RELAY3.IN1
- new net N$20: RELAY3.OUT2, U5.P$1, U5.P$2
- new net N$21: Q3.P$3, RELAY3.ON1
- new net N$22: Q3.P$1, R7.2, R8.2
- new net N$23: D3.1, U5.P$7
- new net N$24: C3.1, D3.3, R9.2, U6.P$4
- new net N$25: J4.2, RELAY4.IN1
- new net N$26: RELAY4.OUT2, U7.P$1, U7.P$2
- new net N$27: Q4.P$3, RELAY4.ON1
- new net N$28: Q4.P$1, R10.2, R11.2
- new net N$29: D4.1, U7.P$7
- new net N$30: C4.1, D4.3, R12.2, U8.P$4
- new net N$9: SV2.1
- net +3V3: now also U3.P$8, U4.P$8, U5.P$8, U6.P$8, U7.P$8, U8.P$1, U8.P$8
- net +5V: now also RELAY2.ON2, RELAY3.ON2, RELAY4.ON2
- net ADDR: now also SV2.5; no longer U2.P$1
- net AGND: now also C2.2, C3.2, C4.2, R12.1, R6.1, R9.1, U4.P$5, U6.P$5, U8.P$5
- net GND: now also Q2.P$2, Q3.P$2, Q4.P$2, R11.1, R5.1, R8.1, U2.P$1, U3.P$5, U4.P$3, U5.P$5, U6.P$3, U7.P$5, U8.P$3
- net N$4: now also J2.3, RELAY2.OUT1; no longer RELAY1.IN2, U1.P$3, U1.P$4
- net SCL: now also SV2.4, U4.P$1, U4.P$10, U6.P$10, U8.P$10
- net SDA: now also SV2.3, U4.P$9, U6.P$1, U6.P$9, U8.P$9
Other:
- board size 100 x 80 mm -> 278.1 x 292.1 mm

Commit message: Added voltage measurement circuitry
Parts:
- removed C2, C3, C4: 1uF, jackIdd:C2.5-2
- removed D2, D3, D4: BAT54, diode:SOT23
- removed J2, J3, J4: 213598-2, con-amp:213598-2
- removed Q2, Q3, Q4: (no value), jackIdd:SOT23
- removed R10, R7: 1K, jackIdd:0411/15
- removed R11, R8: 10K, jackIdd:0411/15
- removed R12, R6, R9: 200K, jackIdd:0411/15
- removed RELAY2, RELAY3, RELAY4: RELAY, iddproject:G5RL-1A-E-HR
- removed U4, U6, U8: ADC, iddproject:ADS1013
- removed U5, U7: Hall Effect, iddproject:ACS711
- R4: value 1K -> 240K
- U2: value ADC -> Current ADC
- U3: value Hall Effect -> Voltage ADC; device iddproject:ACS711 -> iddproject:ADS1013
- moved R5 71.0 mm to (21.6, 6.35)
- moved R4 63.3 mm to (21.6, 10.2)
- moved U3 57.4 mm to (10.2, 10.2)
- moved D1 1.80 mm to (34.3, 69.8)
- moved U1 1.80 mm to (10.2, 57.1)
- moved C1 1.80 mm to (45.7, 68.6)
- moved J1 1.80 mm to (33.0, 31.8)
- moved RELAY1 1.80 mm to (31.8, 55.9)
- moved Q1 1.80 mm to (27.9, 67.3)
- moved R1 1.80 mm to (17.8, 67.3)
- moved R3 1.80 mm to (24.1, 76.2)
- moved SV2 1.80 mm to (63.5, 10.2)
- moved R2 1.80 mm to (40.6, 76.2)
- moved U2 1.80 mm to (40.6, 68.6)
Connections:
- removed net N$11: J2.2, RELAY2.IN1
- removed net N$12: RELAY2.OUT2, U3.P$1, U3.P$2
- removed net N$13: Q2.P$3, RELAY2.ON1
- removed net N$14: Q2.P$1, R4.2, R5.2
- removed net N$15: D2.1, U3.P$7
- removed net N$16: C2.1, D2.3, R6.2, U4.P$4
- removed net N$17: J4.3, RELAY4.OUT1
- removed net N$18: J3.3, RELAY3.OUT1
- removed net N$19: J3.2, RELAY3.IN1
- removed net N$20: RELAY3.OUT2, U5.P$1, U5.P$2
- removed net N$21: Q3.P$3, RELAY3.ON1
- removed net N$22: Q3.P$1, R7.2, R8.2
- removed net N$23: D3.1, U5.P$7
- removed net N$24: C3.1, D3.3, R9.2, U6.P$4
- removed net N$25: J4.2, RELAY4.IN1
- removed net N$26: RELAY4.OUT2, U7.P$1, U7.P$2
- removed net N$27: Q4.P$3, RELAY4.ON1
- removed net N$28: Q4.P$1, R10.2, R11.2
- removed net N$29: D4.1, U7.P$7
- removed net N$30: C4.1, D4.3, R12.2, U8.P$4
- removed net N$4: J2.3, RELAY2.OUT1
- new net N$31: R4.2, R5.2, U3.P$4
- net +3V3: no longer U4.P$8, U5.P$8, U6.P$8, U7.P$8, U8.P$1, U8.P$8
- net +5V: no longer RELAY2.ON2, RELAY3.ON2, RELAY4.ON2
- net AC_LIVE: no longer U3.P$3, U3.P$4, U5.P$3, U5.P$4, U7.P$3, U7.P$4
- net AC_NEUTRAL: no longer RELAY2.IN2, RELAY3.IN2, RELAY4.IN2
- net AGND: no longer C2.2, C3.2, C4.2, R12.1, R6.1, R9.1, U4.P$5, U6.P$5, U8.P$5
- net D10: no longer R7.1
- net D11: no longer U5.P$6
- net D12: no longer R10.1
- net D13: no longer U7.P$6
- net D8: no longer R4.1
- net D9: no longer U3.P$6
- net GND: now also U3.P$3; no longer Q2.P$2, Q3.P$2, Q4.P$2, R11.1, R8.1, U4.P$3, U5.P$5, U6.P$3, U7.P$5, U8.P$3
- net N$3: now also R4.1
- net SCL: now also U3.P$1, U3.P$10; no longer U4.P$1, U4.P$10, U6.P$10, U8.P$10
- net SDA: now also U3.P$9; no longer U4.P$9, U6.P$1, U6.P$9, U8.P$9
Other:
- board size 278.1 x 292.1 mm -> 279.4 x 293.4 mm

Commit message: update
Parts:
- removed J1: 213598-2, con-amp:213598-2
- added +3V3, AC_LIVE, AC_NEUTRAL, GND, OUT+, OUT-: (no value), wirepad:3,81/1,4
- moved R5 73.9 mm to (52.1, 73.7), turned to 180 degrees
- moved U3 71.4 mm to (54.6, 66.0), turned to 180 degrees
- moved R2 64.7 mm to (22.9, 14.0), turned to 180 degrees
- moved R1 60.2 mm to (10.2, 7.62), turned to 90 degrees
- moved R4 57.4 mm to (45.7, 62.2), turned to 90 degrees
- moved R3 52.1 mm to (76.2, 73.7)
- moved Q1 49.9 mm to (15.2, 19.1)
- moved C1 45.7 mm to (91.4, 69.8)
- moved U1 38.6 mm to (48.3, 50.8), turned to 270 degrees
- moved SV2 36.4 mm to (81.3, 41.9), turned to 90 degrees
- moved U2 32.4 mm to (69.8, 54.6), turned to 90 degrees
- moved D1 29.6 mm to (59.7, 54.6)
- moved RELAY1 19.4 mm to (21.6, 39.4), turned to 90 degrees
Connections:
- new net N$4: +3V3.1, U3.P$8
- net +3V3: no longer U3.P$8
- net AC_LIVE: now also AC_LIVE.1
- net AC_NEUTRAL: now also AC_NEUTRAL.1, OUT-.1; no longer RELAY1.IN2
- net GND: now also GND.1; no longer U3.P$5
- net N$1: now also OUT+.1, RELAY1.IN1; no longer J1.3, RELAY1.OUT1
- net N$2: now also RELAY1.OUT1; no longer J1.2, RELAY1.IN1
- net N$31: now also U3.P$5
Routing:
- net AC_NEUTRAL: track 0.00 -> 82.5 mm
- net AC_LIVE: track 0.00 -> 65.1 mm
- net GND: track 0.00 -> 44.4 mm
- net N$3: track 0.00 -> 26.3 mm
- net N$1: track 0.00 -> 23.8 mm
- net N$31: track 0.00 -> 14.1 mm
- net N$6: track 0.00 -> 10.5 mm
- net N$5: track 0.00 -> 7.79 mm

Commit message: adjustments on schematic
Parts:
- added +5V: (no value), wirepad:3,81/1,4
- moved GND 4.02 mm to (21.6, 3.81), turned to 180 degrees
- moved D1 2.54 mm to (59.7, 52.1), turned to 270 degrees
- moved AC_NEUTRAL 1.27 mm to (40.6, 3.81)
- moved SV2 1.27 mm to (81.3, 40.6), turned to 0 degrees
- turned U2 to 270 degrees
Connections:
- removed net +5V: RELAY1.ON2
- new net N$12: +5V.1, RELAY1.ON2
Routing:
- net AC_NEUTRAL: track 82.5 -> 0.00 mm
- net AC_LIVE: track 65.1 -> 1.27 mm
- net GND: track 44.4 -> 0.00 mm
- net N$3: track 26.3 -> 1.76 mm
- net N$1: track 23.8 -> 0.00 mm
- net N$31: track 14.1 -> 0.77 mm
- net N$6: track 10.5 -> 0.00 mm
- net N$5: track 7.79 -> 0.00 mm

Commit message: more schematic?
Parts:
- added C2, C4, C6: 100nF, rcl:C1206
- added C3, C5, C7: .1uF, rcl:C1206
- added C8: 1uF, jackIdd:C2.5-2
- added D2: 1N4004, diode:DO41-10
- added D3: BAT54, diode:SOT23
- added R6: 200K, jackIdd:0411/15
- moved U3 38.1 mm to (85.1, 43.2), turned to 270 degrees
- moved C1 34.3 mm to (57.1, 71.1), turned to 270 degrees
- moved Q1 30.2 mm to (7.62, 48.3), turned to 270 degrees
- moved R2 30.1 mm to (8.89, 40.6)
- moved U1 29.7 mm to (38.1, 78.7)
- moved RELAY1 28.0 mm to (20.3, 67.3)
- moved R1 28.0 mm to (8.89, 35.6), turned to 180 degrees
- moved +3V3 26.8 mm to (90.2, 66.0)
- moved OUT- 25.4 mm to (2.54, 71.1)
- moved OUT+ 25.4 mm to (2.54, 78.7)
- moved R5 23.3 mm to (43.2, 52.1), turned to 270 degrees
- moved D1 22.7 mm to (49.5, 72.4)
- moved R4 21.7 mm to (38.1, 41.9), turned to 0 degrees
- moved SV2 16.6 mm to (82.5, 24.1), turned to 180 degrees
- moved U2 16.1 mm to (74.9, 69.8)
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Connections:
- removed net AGND: C1.2, R3.1, U2.P$5
- removed net N$5 (its old number): Q1.P$3, RELAY1.ON1
- new net N$13: RELAY1.OUT2, U1.P$1, U1.P$2
- new net N$14: C4.2, C5.2, U3.P$3
- new net N$15: C8.1, D3.3, R6.2, U3.P$4
- net +3V3: now also C2.1, C3.1, C6.1, C7.1
- net AC_LIVE: now also R4.1
- net GND: now also C1.2, C2.2, C3.2, C6.2, C7.2, C8.2, R3.1, R6.1, U2.P$5, U3.P$5; no longer U3.P$3
- net N$12: now also D2.C
- net N$3: now also +3V3.1, C4.1, C5.1, U3.P$8; no longer R4.1, RELAY1.OUT2, U1.P$1, U1.P$2
- net N$31: now also D3.1; no longer U3.P$4, U3.P$5
- net N$4: now also D2.A, Q1.P$3, RELAY1.ON1; no longer +3V3.1, U3.P$8
Routing:
- net N$3: track 1.76 -> 0.00 mm
- net AC_LIVE: track 1.27 -> 0.00 mm
- net N$31: track 0.77 -> 0.00 mm
Other:
- board size 279.4 x 293.4 mm -> 109.2 x 86.4 mm

Commit message: update schematic
Parts:
- moved +3V3 33.3 mm to (100.3, 34.3)
- moved C3 21.6 mm to (76.2, 58.4)
- moved C5 18.9 mm to (99.1, 40.6)
- moved U3 16.6 mm to (99.1, 52.1)
- moved C8 15.3 mm to (73.7, 48.3)
- moved D3 14.5 mm to (64.8, 48.3)
- moved C4 14.2 mm to (99.1, 45.7)
- moved R6 13.7 mm to (83.8, 44.5)
- moved C2 11.5 mm to (76.2, 63.5)
- moved R5 8.13 mm to (49.5, 57.1)
- moved R4 6.35 mm to (43.2, 45.7)
Connections:
- removed net N$14: C4.2, C5.2, U3.P$3
- removed net N$3: +3V3.1, C4.1, C5.1, U3.P$8
- net +3V3: now also +3V3.1, C4.1, C5.1, U3.P$8
- net GND: now also C4.2, C5.2, U3.P$3
Routing:
- net GND: track 0.00 -> 163.1 mm
- net SCL: track 0.00 -> 109.9 mm
- net SDA: track 0.00 -> 104.9 mm, vias 0 -> 1
- net D6: track 0.00 -> 89.1 mm, vias 0 -> 1
- net D7: track 0.00 -> 84.1 mm, vias 0 -> 1
- net N$12: track 0.00 -> 64.9 mm
- net +3V3: track 0.00 -> 50.7 mm
- net N$15: track 0.00 -> 32.4 mm
- net N$5: track 0.00 -> 26.9 mm
- net N$31: track 0.00 -> 20.2 mm
- net N$6: track 0.00 -> 18.2 mm
- net N$4: track 0.00 -> 18.0 mm
- net N$7: track 0.00 -> 13.0 mm

Commit message: more layout
Parts:
- moved R4 18.3 mm to (58.4, 35.6)
- moved R5 13.7 mm to (62.2, 52.1)
- moved D1 8.03 mm to (57.1, 69.8)
- moved U1 8.03 mm to (45.7, 76.2)
- moved C6 6.35 mm to (54.6, 78.7)
- moved C1 5.68 mm to (62.2, 68.6)
- moved C7 5.08 mm to (59.7, 78.7)
- moved D3 5.08 mm to (69.8, 48.3)
- moved R3 4.58 mm to (67.3, 63.5)
- moved C8 4.02 mm to (77.5, 49.5)
Routing:
- net AC_NEUTRAL: track 0.00 -> 101.7 mm
- net AC_LIVE: track 0.00 -> 81.0 mm
- net N$13: track 0.00 -> 28.0 mm
- net N$1: track 0.00 -> 14.4 mm
- net N$5: track 26.9 -> 14.8 mm
- net GND: track 163.1 -> 156.3 mm
- net N$12: track 64.9 -> 58.9 mm
- net N$15: track 32.4 -> 27.3 mm
- net D7: track 84.1 -> 81.2 mm
- net +3V3: track 50.7 -> 48.8 mm
- net N$31: track 20.2 -> 21.4 mm
- net N$7: track 13.0 -> 12.0 mm
Other:
- board text added: "TODO: GND"
