File: eagle/schematic/plugstrip.brd (EAGLE design)
At the start: 109.2 x 86.4 mm, 31 parts, among them U1 Hall Effect, U2 Current ADC, U3 Voltage ADC

Commit message: layout!
Parts:
- added F2: (no value), fuse:19560
- added IC1: OPA-SOT23TSV611, linear:SOT23-5
- moved SV2 14.2 mm to (96.3, 20.3), turned to 270 degrees
- moved +3V3 9.40 mm to (100.3, 43.7)
- moved +5V 9.21 mm to (26.7, 12.2)
- moved C5 7.73 mm to (91.4, 39.4)
- moved C4 7.62 mm to (91.4, 45.7)
- moved U3 7.62 mm to (91.4, 52.1)
- moved GND 5.59 mm to (28.4, 3.81)
- moved C6 5.08 mm to (59.7, 78.7)
- moved F1 4.64 mm to (50.0, 11.9), turned to 90 degrees
- moved C7 3.81 mm to (63.5, 78.7)
- moved C1 2.54 mm to (62.2, 71.1), turned to 90 degrees
- moved R5 2.54 mm to (62.2, 54.6)
- moved R4 2.29 mm to (56.1, 35.6)
Connections:
- removed net AC_NEUTRAL: AC_NEUTRAL.1, OUT-.1
- removed net N$2: RELAY1.OUT1
- new net N$17: D3.1, IC1.3, IC1.4
- new net N$3: F1.2, F2.1
- net +3V3: now also IC1.5
- net AC_LIVE: now also F2.2; no longer F1.2
- net GND: now also AC_NEUTRAL.1, IC1.2, OUT-.1
- net N$31: now also IC1.1; no longer D3.1
Routing:
- net GND: track 99.2 -> 498.4 mm, vias 0 -> 4
- net +3V3: track 48.8 -> 220.9 mm, vias 0 -> 2
- net AC_NEUTRAL: track 101.7 -> 0.00 mm
- net D6: track 89.1 -> 147.0 mm, vias 1 -> 0
- net N$17: track 0.00 -> 27.1 mm
- net AC_LIVE: track 71.8 -> 50.6 mm
- net D7: track 81.2 -> 94.3 mm, vias 1 -> 0
- net N$12: track 58.9 -> 48.9 mm
- net N$15: track 27.3 -> 19.9 mm
- net SDA: track 104.9 -> 108.7 mm
- net N$31: track 21.4 -> 18.7 mm
- net N$7: track 12.0 -> 13.4 mm
- net N$13: track 28.0 -> 26.8 mm
- net SCL: track 109.9 -> 111.0 mm
- net N$14: track 12.7 -> 13.2 mm
Other:
- board text removed: "TODO: GND"

Commit message: update board layout
Routing:
- net N$22: track 0.00 -> 35.7 mm
- net N$19: track 0.00 -> 35.7 mm
- net N$8: track 0.00 -> 34.5 mm
- net N$26: track 0.00 -> 34.5 mm
- net N$29: track 0.00 -> 32.0 mm
- net N$2: track 0.00 -> 32.0 mm
- net N$18: track 0.00 -> 29.7 mm
- net N$24: track 0.00 -> 29.7 mm
- net N$23: track 0.00 -> 24.9 mm
- net N$20: track 0.00 -> 24.9 mm
- net N$27: track 0.00 -> 24.6 mm
- net N$11: track 0.00 -> 24.6 mm
- net N$25: track 0.00 -> 22.9 mm
- net N$21: track 0.00 -> 22.9 mm
- net N$28: track 0.00 -> 21.3 mm
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