File: eagle/schematic/plugstrip.sch (EAGLE design)
At the start: 10 parts, among them J1 213598-2, U1 Hall Effect

Commit message: update board
Parts:
- RELAY1: value (none) -> RELAY
- U2: value (none) -> ADC
Changed lines of the file:
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@@
 <parts>
 <part name="U1" library="iddproject" deviceset="ACS711LC" device="" value="Hall Effect"/>
-<part name="RELAY1" library="iddproject" deviceset="G5RL-1A-E-HR" device=""/>
+<part name="RELAY1" library="iddproject" deviceset="G5RL-1A-E-HR" device="" value="RELAY"/>
 <part name="J1" library="con-amp" deviceset="213598-2" device=""/>
 <part name="Q1" library="jackIdd" deviceset="BSH105" device=""/>
@@
 <part name="R3" library="jackIdd" deviceset="R-US_" device="CT14J"/>
 <part name="AGND1" library="supply1" deviceset="AGND" device=""/>
-<part name="U2" library="iddproject" deviceset="ADS1013IDGST" device=""/>
+<part name="U2" library="iddproject" deviceset="ADS1013IDGST" device="" value="ADC"/>
 <part name="+3V2" library="supply1" deviceset="+3V3" device=""/>
 <part name="GND4" library="supply1" deviceset="GND" device=""/>

Commit message: save schematic, board
Parts:
- added C2, C3, C4: 1uF, jackIdd:CSR215E105
- added D2, D3, D4: BAT54, diode:BAT54
- added J2, J3, J4: 213598-2, con-amp:213598-2
- added Q2, Q3, Q4: (no value), jackIdd:BSH105
- added R10, R4, R7: 1K, jackIdd:R-US_CT14J
- added R11, R5, R8: 10K, jackIdd:R-US_CT14J
- added R12, R6, R9: 200K, jackIdd:R-US_CT14J
- added RELAY2, RELAY3, RELAY4: RELAY, iddproject:G5RL-1A-E-HR
- added SV2: (no value), con-lstb:MA13-1
- added U3, U5, U7: Hall Effect, iddproject:ACS711LC
- added U4, U6, U8: ADC, iddproject:ADS1013IDGST
- C1: value (none) -> 1uF
- R3: value (none) -> 200K
Connections:
- removed net D4: R1.1
- removed net D5: U1.FAULT
- new net AC_LIVE: U1.IP-@1, U1.IP-@2, U3.IP-@1, U3.IP-@2, U5.IP-@1, U5.IP-@2, U7.IP-@1, U7.IP-@2
- new net AC_NEUTRAL: RELAY1.IN@2, RELAY2.IN@2, RELAY3.IN@2, RELAY4.IN@2
- new net D10: R7.1, SV2.10
- new net D11: SV2.11, U5.FAULT
- new net D12: R10.1, SV2.12
- new net D13: SV2.13, U7.FAULT
- new net D6: R1.1, SV2.6
- new net D7: SV2.7, U1.FAULT
- new net D8: R4.1, SV2.8
- new net D9: SV2.9, U3.FAULT
- new net N$10: SV2.2
- new net N$11: J2.2, RELAY2.IN@1
- new net N$12: RELAY2.OUT@2, U3.IP+@1, U3.IP+@2
- new net N$13: Q2.D, RELAY2.ON@1
- new net N$14: Q2.G, R4.2, R5.2
- new net N$15: D2.A, U3.VIOUT
- new net N$16: C2.1, D2.C, R6.2, U4.AIN0
- new net N$17: J4.3, RELAY4.OUT@1
- new net N$18: J3.3, RELAY3.OUT@1
- new net N$19: J3.2, RELAY3.IN@1
- new net N$20: RELAY3.OUT@2, U5.IP+@1, U5.IP+@2
- new net N$21: Q3.D, RELAY3.ON@1
- new net N$22: Q3.G, R7.2, R8.2
- new net N$23: D3.A, U5.VIOUT
- new net N$24: C3.1, D3.C, R9.2, U6.AIN0
- new net N$25: J4.2, RELAY4.IN@1
- new net N$26: RELAY4.OUT@2, U7.IP+@1, U7.IP+@2
- new net N$27: Q4.D, RELAY4.ON@1
- new net N$28: Q4.G, R10.2, R11.2
- new net N$29: D4.A, U7.VIOUT
- new net N$30: C4.1, D4.C, R12.2, U8.AIN0
- new net N$9: SV2.1
- net +3V3: now also U3.VCC, U4.VDD, U5.VCC, U6.VDD, U7.VCC, U8.ADDR, U8.VDD
- net +5V: now also RELAY2.ON@2, RELAY3.ON@2, RELAY4.ON@2
- net ADDR: now also SV2.5; no longer U2.ADDR
- net AGND: now also C2.2, C3.2, C4.2, R12.1, R6.1, R9.1, U4.AIN1, U6.AIN1, U8.AIN1
- net GND: now also Q2.S, Q3.S, Q4.S, R11.1, R5.1, R8.1, U2.ADDR, U3.GND, U4.GND, U5.GND, U6.GND, U7.GND, U8.GND
- net N$4: now also J2.3, RELAY2.OUT@1; no longer RELAY1.IN@2, U1.IP-@1, U1.IP-@2
- net SCL: now also SV2.4, U4.ADDR, U4.SCL, U6.SCL, U8.SCL
- net SDA: now also SV2.3, U4.SDA, U6.ADDR, U6.SDA, U8.SDA
Other:
- moved on the sheet: C1, D1, J1, Q1, R1, R2, R3, RELAY1, U1, U2

Commit message: Added voltage measurement circuitry
Parts:
- removed C2, C3, C4: 1uF, jackIdd:CSR215E105
- removed D2, D3, D4: BAT54, diode:BAT54
- removed J2, J3, J4: 213598-2, con-amp:213598-2
- removed Q2, Q3, Q4: (no value), jackIdd:BSH105
- removed R10, R7: 1K, jackIdd:R-US_CT14J
- removed R11, R8: 10K, jackIdd:R-US_CT14J
- removed R12, R6, R9: 200K, jackIdd:R-US_CT14J
- removed RELAY2, RELAY3, RELAY4: RELAY, iddproject:G5RL-1A-E-HR
- removed U4, U6, U8: ADC, iddproject:ADS1013IDGST
- removed U5, U7: Hall Effect, iddproject:ACS711LC
- R4: value 1K -> 240K; device jackIdd:R-US_CT14J -> jackIdd:R-US_0411/15
- R5: device jackIdd:R-US_CT14J -> jackIdd:R-US_0411/15
- U2: value ADC -> Current ADC
- U3: value Hall Effect -> Voltage ADC; device iddproject:ACS711LC -> iddproject:ADS1013IDGST
Connections:
- removed net N$11: J2.2, RELAY2.IN@1
- removed net N$12: RELAY2.OUT@2, U3.IP+@1, U3.IP+@2
- removed net N$13: Q2.D, RELAY2.ON@1
- removed net N$14: Q2.G, R4.2, R5.2
- removed net N$15: D2.A, U3.VIOUT
- removed net N$16: C2.1, D2.C, R6.2, U4.AIN0
- removed net N$17: J4.3, RELAY4.OUT@1
- removed net N$18: J3.3, RELAY3.OUT@1
- removed net N$19: J3.2, RELAY3.IN@1
- removed net N$20: RELAY3.OUT@2, U5.IP+@1, U5.IP+@2
- removed net N$21: Q3.D, RELAY3.ON@1
- removed net N$22: Q3.G, R7.2, R8.2
- removed net N$23: D3.A, U5.VIOUT
- removed net N$24: C3.1, D3.C, R9.2, U6.AIN0
- removed net N$25: J4.2, RELAY4.IN@1
- removed net N$26: RELAY4.OUT@2, U7.IP+@1, U7.IP+@2
- removed net N$27: Q4.D, RELAY4.ON@1
- removed net N$28: Q4.G, R10.2, R11.2
- removed net N$29: D4.A, U7.VIOUT
- removed net N$30: C4.1, D4.C, R12.2, U8.AIN0
- removed net N$4: J2.3, RELAY2.OUT@1
- new net N$31: R4.2, R5.2, U3.AIN0
- net +3V3: now also U3.VDD; no longer U3.VCC, U4.VDD, U5.VCC, U6.VDD, U7.VCC, U8.ADDR, U8.VDD
- net +5V: no longer RELAY2.ON@2, RELAY3.ON@2, RELAY4.ON@2
- net AC_LIVE: no longer U3.IP-@1, U3.IP-@2, U5.IP-@1, U5.IP-@2, U7.IP-@1, U7.IP-@2
- net AC_NEUTRAL: no longer RELAY2.IN@2, RELAY3.IN@2, RELAY4.IN@2
- net AGND: no longer C2.2, C3.2, C4.2, R12.1, R6.1, R9.1, U4.AIN1, U6.AIN1, U8.AIN1
- net D10: no longer R7.1
- net D11: no longer U5.FAULT
- net D12: no longer R10.1
- net D13: no longer U7.FAULT
- net D8: no longer R4.1
- net D9: no longer U3.FAULT
- net GND: now also U3.AIN1; no longer Q2.S, Q3.S, Q4.S, R11.1, R8.1, U4.GND, U5.GND, U6.GND, U7.GND, U8.GND
- net N$3: now also R4.1
- net SCL: now also U3.ADDR, U3.SCL; no longer U4.ADDR, U4.SCL, U6.SCL, U8.SCL
- net SDA: now also U3.SDA; no longer U4.SDA, U6.ADDR, U6.SDA, U8.SDA
Other:
- moved on the sheet: C1, D1, J1, Q1, R1, R2, R3, R4, R5, RELAY1, SV2, U1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

Commit message: update
Parts:
- removed J1: 213598-2, con-amp:213598-2
- added +3V3, AC_LIVE, AC_NEUTRAL, GND, OUT+, OUT-: (no value), wirepad:3,81/1,4
Connections:
- new net N$4: +3V3.P, U3.VDD
- net +3V3: no longer U3.VDD
- net AC_LIVE: now also AC_LIVE.P
- net AC_NEUTRAL: now also AC_NEUTRAL.P, OUT-.P; no longer RELAY1.IN@2
- net GND: now also GND.P; no longer U3.AIN1
- net N$1: now also OUT+.P, RELAY1.IN@1; no longer J1.3, RELAY1.OUT@1
- net N$2: now also RELAY1.OUT@1; no longer J1.2, RELAY1.IN@1
- net N$31: now also U3.AIN1
Changed lines of the file:
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@@
 <part name="U1" library="iddproject" deviceset="ACS711LC" device="" value="Hall Effect"/>
 <part name="RELAY1" library="iddproject" deviceset="G5RL-1A-E-HR" device="" value="RELAY"/>
-<part name="J1" library="con-amp" deviceset="213598-2" device=""/>
 <part name="Q1" library="jackIdd" deviceset="BSH105" device=""/>
 <part name="R1" library="jackIdd" deviceset="R-US_" device="CT14J" value="1K"/>
@@
 <part name="GND17" library="supply1" deviceset="GND" device=""/>
 <part name="U3" library="iddproject" deviceset="ADS1013IDGST" device="" value="Voltage ADC"/>
-<part name="+3V9" library="supply1" deviceset="+3V3" device=""/>
-<part name="GND19" library="supply1" deviceset="GND" device=""/>
+<part name="OUT+" library="wirepad" deviceset="3,81/1,4" device=""/>
+<part name="OUT-" library="wirepad" deviceset="3,81/1,4" device=""/>
+<part name="+3V3" library="wirepad" deviceset="3,81/1,4" device=""/>
+<part name="GND" library="wirepad" deviceset="3,81/1,4" device=""/>
+<part name="AC_LIVE" library="wirepad" deviceset="3,81/1,4" device=""/>
+<part name="AC_NEUTRAL" library="wirepad" deviceset="3,81/1,4" device=""/>
 </parts>
 <sheets>
@@
 <instance part="U1" gate="G$1" x="0" y="0"/>
 <instance part="RELAY1" gate="G$1" x="-58.42" y="-20.32" rot="R90"/>
-<instance part="J1" gate="G$1" x="-93.98" y="0" rot="R180"/>
 <instance part="Q1" gate="G$1" x="-81.28" y="-60.96"/>
 <instance part="R1" gate="G$1" x="-114.3" y="-60.96"/>
@@
 <instance part="GND17" gate="1" x="-30.48" y="58.42" rot="R180"/>
 <instance part="U3" gate="G$1" x="15.24" y="38.1"/>
-<instance part="+3V9" gate="G$1" x="63.5" y="38.1" rot="R270"/>
-<instance part="GND19" gate="1" x="-10.16" y="25.4"/>
+<instance part="OUT+" gate="1" x="-104.14" y="5.08"/>
+<instance part="OUT-" gate="1" x="-104.14" y="-5.08"/>
+<instance part="+3V3" gate="1" x="73.66" y="38.1" rot="R180"/>
+<instance part="GND" gate="1" x="-68.58" y="-81.28" rot="R180"/>
+<instance part="AC_LIVE" gate="1" x="60.96" y="-27.94" rot="R180"/>
+<instance part="AC_NEUTRAL" gate="1" x="60.96" y="-38.1" rot="R180"/>
 </instances>
 <busses>
 </busses>
 <nets>
-<net name="N$1" class="1">
-<segment>
-<pinref part="J1" gate="G$1" pin="3"/>
-<wire x1="-91.44" y1="2.54" x2="-78.74" y2="2.54" width="0.1524" layer="91"/>
-<wire x1="-78.74" y1="2.54" x2="-78.74" y2="5.08" width="0.1524" layer="91"/>
-<pinref part="RELAY1" gate="G$1" pin="OUT@1"/>
-<wire x1="-78.74" y1="5.08" x2="-71.12" y2="5.08" width="0.1524" layer="91"/>
-</segment>
-</net>
-<net name="N$2" class="1">
-<segment>
-<pinref part="J1" gate="G$1" pin="2"/>
-<wire x1="-91.44" y1="0" x2="-78.74" y2="0" width="0.1524" layer="91"/>
-<wire x1="-78.74" y1="0" x2="-78.74" y2="-5.08" width="0.1524" layer="91"/>
-<pinref part="RELAY1" gate="G$1" pin="IN@1"/>
-<wire x1="-78.74" y1="-5.08" x2="-71.12" y2="-5.08" width="0.1524" layer="91"/>
-</segment>
-</net>
-<net name="N$3" class="0">
+<net name="N$3" class="1">
 <segment>
 <pinref part="RELAY1" gate="G$1" pin="OUT@2"/>
@@
 <pinref part="GND2" gate="1" pin="GND"/>
 <wire x1="-81.28" y1="-73.66" x2="-81.28" y2="-78.74" width="0.1524" layer="91"/>
+<pinref part="GND" gate="1" pin="P"/>
+<wire x1="-81.28" y1="-78.74" x2="-71.12" y2="-78.74" width="0.1524" layer="91"/>
+<wire x1="-71.12" y1="-78.74" x2="-71.12" y2="-81.28" width="0.1524" layer="91"/>
+<junction x="-81.28" y="-78.74"/>
 </segment>
 <segment>
@@
 <junction x="-30.48" y="53.34"/>
 </segment>
-<segment>
-<pinref part="U3" gate="G$1" pin="AIN1"/>
-<wire x1="-5.08" y1="33.02" x2="-10.16" y2="33.02" width="0.1524" layer="91"/>
-<wire x1="-10.16" y1="33.02" x2="-10.16" y2="27.94" width="0.1524" layer="91"/>
-<pinref part="GND19" gate="1" pin="GND"/>
-</segment>
 </net>
 <net name="+5V" class="0">
@@
 <pinref part="U2" gate="G$1" pin="VDD"/>
 <wire x1="137.16" y1="-2.54" x2="121.92" y2="-2.54" width="0.1524" layer="91"/>
-</segment>
-<segment>
-<pinref part="U3" gate="G$1" pin="VDD"/>
-<wire x1="35.56" y1="38.1" x2="60.96" y2="38.1" width="0.1524" layer="91"/>
-<pinref part="+3V9" gate="G$1" pin="+3V3"/>
 </segment>
 </net>
@@
 <junction x="-22.86" y="-5.08"/>
 <wire x1="-27.94" y1="-5.08" x2="-27.94" y2="-27.94" width="0.1524" layer="91"/>
-<wire x1="-27.94" y1="-27.94" x2="30.48" y2="-27.94" width="0.1524" layer="91"/>
-<label x="30.48" y="-27.94" size="1.778" layer="95"/>
+<wire x1="-27.94" y1="-27.94" x2="58.42" y2="-27.94" width="0.1524" layer="91"/>
+<pinref part="AC_LIVE" gate="1" pin="P"/>
 </segment>
 </net>
 <net name="AC_NEUTRAL" class="1">
 <segment>
-<pinref part="RELAY1" gate="G$1" pin="IN@2"/>
-<wire x1="-38.1" y1="-5.08" x2="-33.02" y2="-5.08" width="0.1524" layer="91"/>
-<wire x1="-33.02" y1="-5.08" x2="-33.02" y2="-30.48" width="0.1524" layer="91"/>
-<wire x1="-33.02" y1="-30.48" x2="38.1" y2="-30.48" width="0.1524" layer="91"/>
-<label x="38.1" y="-30.48" size="1.778" layer="95"/>
+<pinref part="OUT-" gate="1" pin="P"/>
+<wire x1="-101.6" y1="-5.08" x2="-86.36" y2="-5.08" width="0.1524" layer="91"/>
+<wire x1="-86.36" y1="-5.08" x2="-86.36" y2="-17.78" width="0.1524" layer="91"/>
+<wire x1="-86.36" y1="-17.78" x2="-33.02" y2="-17.78" width="0.1524" layer="91"/>
+<wire x1="-33.02" y1="-17.78" x2="-33.02" y2="-33.02" width="0.1524" layer="91"/>
+<wire x1="-33.02" y1="-33.02" x2="15.24" y2="-33.02" width="0.1524" layer="91"/>
+<wire x1="15.24" y1="-33.02" x2="15.24" y2="-38.1" width="0.1524" layer="91"/>
+<pinref part="AC_NEUTRAL" gate="1" pin="P"/>
+<wire x1="15.24" y1="-38.1" x2="58.42" y2="-38.1" width="0.1524" layer="91"/>
 </segment>
 </net>
@@
 <pinref part="R4" gate="G$1" pin="2"/>
 <pinref part="R5" gate="G$1" pin="2"/>
-<wire x1="-30.48" y1="30.48" x2="-30.48" y2="35.56" width="0.1524" layer="91"/>
+<wire x1="-30.48" y1="30.48" x2="-30.48" y2="33.02" width="0.1524" layer="91"/>
 <pinref part="U3" gate="G$1" pin="AIN0"/>
+<wire x1="-30.48" y1="33.02" x2="-30.48" y2="35.56" width="0.1524" layer="91"/>
 <wire x1="-30.48" y1="35.56" x2="-30.48" y2="38.1" width="0.1524" layer="91"/>
 <wire x1="-5.08" y1="35.56" x2="-30.48" y2="35.56" width="0.1524" layer="91"/>
 <junction x="-30.48" y="35.56"/>
-</segment>
-</net>
+<pinref part="U3" gate="G$1" pin="AIN1"/>
+<wire x1="-5.08" y1="33.02" x2="-30.48" y2="33.02" width="0.1524" layer="91"/>
+<junction x="-30.48" y="33.02"/>
+</segment>
+</net>
+<net name="N$4" class="0">
+<segment>
+<pinref part="U3" gate="G$1" pin="VDD"/>
+<wire x1="35.56" y1="38.1" x2="71.12" y2="38.1" width="0.1524" layer="91"/>
+<pinref part="+3V3" gate="1" pin="P"/>
+</segment>
+</net>
+<net name="N$1" class="0">
+<segment>
+<pinref part="RELAY1" gate="G$1" pin="IN@1"/>
+<wire x1="-71.12" y1="-5.08" x2="-81.28" y2="-5.08" width="0.1524" layer="91"/>
+<wire x1="-81.28" y1="-5.08" x2="-91.44" y2="5.08" width="0.1524" layer="91"/>
+<pinref part="OUT+" gate="1" pin="P"/>
+<wire x1="-91.44" y1="5.08" x2="-101.6" y2="5.08" width="0.1524" layer="91"/>
+</segment>
+</net>
+<net name="N$2" class="0">
+<segment>
+<pinref part="RELAY1" gate="G$1" pin="OUT@1"/>
+<wire x1="-71.12" y1="5.08" x2="-43.18" y2="5.08" width="0.1524" layer="91"/>
+</segment>
+</net>
+<net name="N$11" class="0">
+<segment>
+<wire x1="-43.18" y1="-5.08" x2="-66.04" y2="-5.08" width="0.1524" layer="91"/>
+</segment>
+</net>

Commit message: adjustments on schematic
Parts:
- added +5V: (no value), wirepad:3,81/1,4
Connections:
- removed net +5V: RELAY1.ON@2
- new net N$12: +5V.P, RELAY1.ON@2
Other:
- moved on the sheet: SV2
Changed lines of the file:
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@@
 <classes>
 <class number="0" name="default" width="0.4064" drill="0">
+<clearance class="0" value="0.3048"/>
 </class>
-<class number="1" name="analoghot" width="2.54" drill="0">
+<class number="1" name="analoghot" width="4.5974" drill="0">
+<clearance class="1" value="0.6096"/>
 </class>
 </classes>
@@
 <part name="GND2" library="supply1" deviceset="GND" device=""/>
 <part name="GND3" library="supply1" deviceset="GND" device=""/>
-<part name="P+1" library="supply1" deviceset="+5V" device=""/>
 <part name="+3V1" library="supply1" deviceset="+3V3" device=""/>
 <part name="D1" library="diode" deviceset="BAT54" device=""/>
@@
 <part name="AC_LIVE" library="wirepad" deviceset="3,81/1,4" device=""/>
 <part name="AC_NEUTRAL" library="wirepad" deviceset="3,81/1,4" device=""/>
+<part name="+5V" library="wirepad" deviceset="3,81/1,4" device=""/>
 </parts>
 <sheets>
@@
 <instance part="GND2" gate="1" x="-81.28" y="-81.28"/>
 <instance part="GND3" gate="1" x="17.78" y="-15.24"/>
-<instance part="P+1" gate="1" x="-35.56" y="-48.26" rot="R90"/>
 <instance part="+3V1" gate="G$1" x="25.4" y="7.62" rot="R270"/>
 <instance part="D1" gate="G$1" x="38.1" y="2.54"/>
@@
 <instance part="+3V2" gate="G$1" x="139.7" y="-2.54" rot="R270"/>
 <instance part="GND4" gate="1" x="76.2" y="10.16" rot="R180"/>
-<instance part="SV2" gate="G$1" x="-167.64" y="-15.24"/>
+<instance part="SV2" gate="G$1" x="-111.76" y="-30.48"/>
 <instance part="R4" gate="G$1" x="-30.48" y="25.4" rot="R90"/>
 <instance part="R5" gate="G$1" x="-30.48" y="43.18" rot="R270"/>
@@
 <instance part="AC_LIVE" gate="1" x="60.96" y="-27.94" rot="R180"/>
 <instance part="AC_NEUTRAL" gate="1" x="60.96" y="-38.1" rot="R180"/>
+<instance part="+5V" gate="1" x="-20.32" y="-50.8" rot="R180"/>
 </instances>
 <busses>
@@
 </segment>
 </net>
-<net name="+5V" class="0">
-<segment>
-<pinref part="RELAY1" gate="G$1" pin="ON@2"/>
-<pinref part="P+1" gate="1" pin="+5V"/>
-<wire x1="-38.1" y1="-35.56" x2="-33.02" y2="-35.56" width="0.1524" layer="91"/>
-<wire x1="-33.02" y1="-35.56" x2="-33.02" y2="-48.26" width="0.1524" layer="91"/>
-</segment>
-</net>
 <net name="+3V3" class="0">
 <segment>
@@
 <segment>
 <pinref part="SV2" gate="G$1" pin="4"/>
-<wire x1="-160.02" y1="-22.86" x2="-152.4" y2="-22.86" width="0.1524" layer="91"/>
-<label x="-154.94" y="-22.86" size="1.778" layer="95"/>
+<wire x1="-104.14" y1="-38.1" x2="-96.52" y2="-38.1" width="0.1524" layer="91"/>
+<label x="-99.06" y="-38.1" size="1.778" layer="95"/>
 </segment>
 <segment>
@@
 <segment>
 <pinref part="SV2" gate="G$1" pin="3"/>
-<wire x1="-160.02" y1="-25.4" x2="-152.4" y2="-25.4" width="0.1524" layer="91"/>
-<label x="-154.94" y="-25.4" size="1.778" layer="95"/>
+<wire x1="-104.14" y1="-40.64" x2="-96.52" y2="-40.64" width="0.1524" layer="91"/>
+<label x="-99.06" y="-40.64" size="1.778" layer="95"/>
 </segment>
 <segment>
@@
 <segment>
 <pinref part="SV2" gate="G$1" pin="5"/>
-<wire x1="-160.02" y1="-20.32" x2="-152.4" y2="-20.32" width="0.1524" layer="91"/>
-<label x="-154.94" y="-20.32" size="1.778" layer="95"/>
+<wire x1="-104.14" y1="-35.56" x2="-96.52" y2="-35.56" width="0.1524" layer="91"/>
+<label x="-99.06" y="-35.56" size="1.778" layer="95"/>
 </segment>
 </net>
@@
 <segment>
 <pinref part="SV2" gate="G$1" pin="1"/>
-<wire x1="-160.02" y1="-30.48" x2="-152.4" y2="-30.48" width="0.1524" layer="91"/>
+<wire x1="-104.14" y1="-45.72" x2="-96.52" y2="-45.72" width="0.1524" layer="91"/>
 </segment>
 </net>
@@
 <segment>
 <pinref part="SV2" gate="G$1" pin="2"/>
-<wire x1="-160.02" y1="-27.94" x2="-152.4" y2="-27.94" width="0.1524" layer="91"/>
+<wire x1="-104.14" y1="-43.18" x2="-96.52" y2="-43.18" width="0.1524" layer="91"/>
 </segment>
 </net>
@@
 <segment>
 <pinref part="SV2" gate="G$1" pin="6"/>
-<wire x1="-160.02" y1="-17.78" x2="-152.4" y2="-17.78" width="0.1524" layer="91"/>
-<label x="-154.94" y="-17.78" size="1.778" layer="95"/>
+<wire x1="-104.14" y1="-33.02" x2="-96.52" y2="-33.02" width="0.1524" layer="91"/>
+<label x="-99.06" y="-33.02" size="1.778" layer="95"/>
 </segment>
 <segment>
@@
 <segment>
 <pinref part="SV2" gate="G$1" pin="8"/>
-<wire x1="-160.02" y1="-12.7" x2="-152.4" y2="-12.7" width="0.1524" layer="91"/>
-<label x="-154.94" y="-12.7" size="1.778" layer="95"/>
+<wire x1="-104.14" y1="-27.94" x2="-96.52" y2="-27.94" width="0.1524" layer="91"/>
+<label x="-99.06" y="-27.94" size="1.778" layer="95"/>
 </segment>
 </net>
@@
 <segment>
 <pinref part="SV2" gate="G$1" pin="9"/>
-<wire x1="-160.02" y1="-10.16" x2="-152.4" y2="-10.16" width="0.1524" layer="91"/>
-<label x="-154.94" y="-10.16" size="1.778" layer="95"/>
+<wire x1="-104.14" y1="-25.4" x2="-96.52" y2="-25.4" width="0.1524" layer="91"/>
+<label x="-99.06" y="-25.4" size="1.778" layer="95"/>
 </segment>
 </net>
@@
 <segment>
 <pinref part="SV2" gate="G$1" pin="10"/>
-<wire x1="-160.02" y1="-7.62" x2="-152.4" y2="-7.62" width="0.1524" layer="91"/>
-<label x="-154.94" y="-7.62" size="1.778" layer="95"/>
+<wire x1="-104.14" y1="-22.86" x2="-96.52" y2="-22.86" width="0.1524" layer="91"/>
+<label x="-99.06" y="-22.86" size="1.778" layer="95"/>
 </segment>
 </net>
@@
 <segment>
 <pinref part="SV2" gate="G$1" pin="11"/>
-<wire x1="-160.02" y1="-5.08" x2="-152.4" y2="-5.08" width="0.1524" layer="91"/>
-<label x="-154.94" y="-5.08" size="1.778" layer="95"/>
+<wire x1="-104.14" y1="-20.32" x2="-96.52" y2="-20.32" width="0.1524" layer="91"/>
+<label x="-99.06" y="-20.32" size="1.778" layer="95"/>
 </segment>
 </net>
@@
 <segment>
 <pinref part="SV2" gate="G$1" pin="12"/>
-<wire x1="-160.02" y1="-2.54" x2="-152.4" y2="-2.54" width="0.1524" layer="91"/>
-<label x="-154.94" y="-2.54" size="1.778" layer="95"/>
+<wire x1="-104.14" y1="-17.78" x2="-96.52" y2="-17.78" width="0.1524" layer="91"/>
+<label x="-99.06" y="-17.78" size="1.778" layer="95"/>
 </segment>
 </net>
@@
 <segment>
 <pinref part="SV2" gate="G$1" pin="13"/>
-<wire x1="-160.02" y1="0" x2="-152.4" y2="0" width="0.1524" layer="91"/>
-<label x="-154.94" y="0" size="1.778" layer="95"/>
+<wire x1="-104.14" y1="-15.24" x2="-96.52" y2="-15.24" width="0.1524" layer="91"/>
+<label x="-99.06" y="-15.24" size="1.778" layer="95"/>
 </segment>
 </net>
@@
 <segment>
 <pinref part="SV2" gate="G$1" pin="7"/>
-<wire x1="-160.02" y1="-15.24" x2="-152.4" y2="-15.24" width="0.1524" layer="91"/>
-<label x="-154.94" y="-15.24" size="1.778" layer="95"/>
+<wire x1="-104.14" y1="-30.48" x2="-96.52" y2="-30.48" width="0.1524" layer="91"/>
+<label x="-99.06" y="-30.48" size="1.778" layer="95"/>
 </segment>
 </net>
@@
 </segment>
 </net>
+<net name="N$12" class="0">
+<segment>
+<pinref part="RELAY1" gate="G$1" pin="ON@2"/>
+<wire x1="-38.1" y1="-35.56" x2="-33.02" y2="-35.56" width="0.1524" layer="91"/>
+<wire x1="-33.02" y1="-35.56" x2="-33.02" y2="-50.8" width="0.1524" layer="91"/>
+<pinref part="+5V" gate="1" pin="P"/>
+<wire x1="-33.02" y1="-50.8" x2="-22.86" y2="-50.8" width="0.1524" layer="91"/>
+</segment>
+</net>

Commit message: more schematic?
Parts:
- added C2, C4, C6: 100nF, rcl:C-USC1206
- added C3, C5, C7: .1uF, rcl:C-USC1206
- added C8: 1uF, jackIdd:CSR215E105
- added D2: 1N4004, diode:1N4004
- added D3: BAT54, diode:BAT54
- added R6: 200K, jackIdd:R-US_CT14J
Connections:
- removed net AGND: C1.2, R3.1, U2.AIN1
- removed net N$5 (its old number): Q1.D, RELAY1.ON@1
- new net N$13: RELAY1.OUT@2, U1.IP+@1, U1.IP+@2
- new net N$14: C4.2, C5.2, U3.GND
- new net N$15: C8.1, D3.C, R6.2, U3.AIN0
- net +3V3: now also C2.1, C3.1, C6.1, C7.1
- net AC_LIVE: now also R4.1
- net GND: now also C1.2, C2.2, C3.2, C6.2, C7.2, C8.2, R3.1, R6.1, U2.AIN1, U3.AIN1; no longer U3.GND
- net N$12: now also D2.C
- net N$3: now also +3V3.P, C4.1, C5.1, U3.VDD; no longer R4.1, RELAY1.OUT@2, U1.IP+@1, U1.IP+@2
- net N$31: now also D3.A; no longer U3.AIN0, U3.AIN1
- net N$4: now also D2.A, Q1.D, RELAY1.ON@1; no longer +3V3.P, U3.VDD
Other:
- moved on the sheet: +3V3, AC_LIVE, AC_NEUTRAL, C1, D1, R3, R4, R5, U1, U2, U3
